Commit message: Updated sick_lms1xx.urdf.xacro: turned gravity ON.

File: urdf/sick_lms1xx.urdf.xacro (robot description, xacro)
@@ -30,10 +30,11 @@
     <link name="${frame}">
       <inertial>
-        <mass value="1.1" />
+        <!--mass value="1.1" /-->
+        <mass value="0.0001" />
         <origin xyz="0 0 0" />
         <inertia ixx="${0.0833333 * 1.1 * (0.102*0.102 + 0.152*0.152)}" ixy="0.0" ixz="0.0"
           iyy="${0.0833333 * 1.1 * (0.105*0.105 + 0.152*0.152)}" iyz="0.0"
           izz="${0.0833333 * 1.1 * (0.105*0.105 + 0.102*0.102)}" />
-      </inertial>
+        </inertial>
       <visual>
         <origin xyz="0 0 0" rpy="0 0 0" />
@@ -51,6 +52,6 @@
     </link>
     <gazebo reference="${frame}">
-      <turnGravityOff>true</turnGravityOff>
-      <sensor type="ray" name="${frame}">
+      <turnGravityOff>false</turnGravityOff>
+      <sensor type="gpu_ray" name="${frame}">
         <pose>0 0 0 0 0 0</pose>
         <visualize>false</visualize>
@@ -76,5 +77,5 @@
           </noise>
         </ray>
-        <plugin name="gazebo_ros_laser" filename="libgazebo_ros_laser.so">
+        <plugin name="gazebo_ros_laser" filename="libgazebo_ros_gpu_laser.so">
           <topicName>${topic}</topicName>
           <frameName>${frame}</frameName>
